Commit message: 模型修改

File: mybot_description/urdf/arm_gazebo.xacro (robot description, xacro)
@@ -1,4 +1,5 @@
 <?xml version="1.0"?>
 <robot name="six_arm" xmlns:xacro="http://www.ros.org/wiki/xacro">
+    <!-- <xacro:include filename="./arm.xacro" /> -->
     <xacro:include filename="$(find mybot_description)/urdf/arm.xacro" />
     <!-- /////////////////////////////////   Gazebo   ////////////////////////////////////// -->

File: mybot_description/urdf/large_base_gazebo.xacro (robot description, xacro)
@@ -1,87 +1,8 @@
 <?xml version="1.0"?>
-<robot name="originbot"
-    xmlns:xacro="http://www.ros.org/wiki/xacro">
-    <!-- 大号机器人模型 -->
-    <!-- PROPERTY LIST -->
-    <xacro:property name="M_PI" value="3.1415926"/>
-    <xacro:property name="base_mass" value="2" />
-    <xacro:property name="base_radius" value="0.3"/>
-    <xacro:property name="base_width" value="0.370"/>
-    <xacro:property name="base_length" value="0.370"/>
-    <xacro:property name="base_height" value="0.260"/>
-    <!-- 轮子 -->
-    <xacro:property name="wheel_mass" value="0.4" />
-    <xacro:property name="wheel_radius" value="0.065"/>
-    <xacro:property name="wheel_length" value="0.050"/>
-    <xacro:property name="wheel_joint_x" value="0.04"/>
-    <xacro:property name="wheel_joint_y" value="0.38"/>
-    <xacro:property name="wheel_joint_z" value="0.105"/>
-    <!-- 支撑轮 -->
-    <xacro:property name="caster_mass" value="0.4" />
-    <xacro:property name="caster_radius" value="0.02"/>
-    <!-- wheel_radius - ( base_length/2 - wheel_joint_z) -->
-    <xacro:property name="caster_joint_x" value="0.10"/>
-    <!-- Defining the colors used in this robot -->
-    <material name="yellow">
-        <color rgba="1 0.4 0 1"/>
-    </material>
-    <material name="black">
-        <color rgba="0 0 0 0.95"/>
-    </material>
-    <material name="gray">
-        <color rgba="0.75 0.75 0.75 1"/>
-    </material>
-    <!-- Macro for inertia matrix -->
-    <!-- 球面惯性矩阵 -->
-    <xacro:macro name="sphere_inertial_matrix" params="m r">
-        <inertial>
-            <mass value="${m}" />
-            <inertia ixx="${2*m*r*r/5}" ixy="0" ixz="0" iyy="${2*m*r*r/5}" iyz="0" izz="${2*m*r*r/5}" />
-        </inertial>
-    </xacro:macro>
-    <!-- 圆柱惯性矩阵 -->
-    <xacro:macro name="cylinder_inertial_matrix" params="m r h">
-        <inertial>
-            <mass value="${m}" />
-            <inertia ixx="${m*(3*r*r+h*h)/12}" ixy = "0" ixz = "0" iyy="${m*(3*r*r+h*h)/12}" iyz = "0" izz="${m*r*r/2}" />
-        </inertial>
-    </xacro:macro>
-    <!-- 方块惯性矩阵 -->
-    <xacro:macro name="box_inertial_matrix" params="m l w h">
-        <inertial>
-            <mass value="${m}" />
-            <inertia ixx="${m*(h*h + l*l)/12}" ixy = "0" ixz = "0" iyy="${m*(w*w + l*l)/12}" iyz= "0" izz="${m*(w*w + h*h)/12}" />
-        </inertial>
-    </xacro:macro>
-    <!-- Macro for robot 轮子 -->
-    <xacro:macro name="wheel" params="prefix reflect">
-        <joint name="${prefix}_wheel_joint" type="continuous">
-            <origin xyz="${wheel_joint_x} ${reflect*(base_width+wheel_length)/2} ${-wheel_joint_z}" rpy="0 0 0"/>
-            <parent link="base_link"/>
-            <child link="${prefix}_wheel_link"/>
-            <axis xyz="0 1 0"/>
-        </joint>
-        <link name="${prefix}_wheel_link">
-            <visual>
-                <origin xyz="0 0 0" rpy="${M_PI/2} 0 0" />
-                <geometry>
-                    <cylinder radius="${wheel_radius}" length = "${wheel_length}"/>
-                </geometry>
-                <material name="gray" />
-            </visual>
-            <collision>
-                <origin xyz="0 0 0" rpy="${M_PI/2} 0 0" />
-                <geometry>
-                    <cylinder radius="${wheel_radius}" length = "${wheel_length}"/>
-                </geometry>
-            </collision>
-            <xacro:cylinder_inertial_matrix m="${wheel_mass}" r="${wheel_radius}" h="${wheel_length}" />
-        </link>
-        <gazebo reference="${prefix}_wheel_link">
-            <material>Gazebo/Gray</material>
-            <mu1>100000.0</mu1>
-            <mu2>100000.0</mu2>
-        </gazebo>
-        <!-- Transmission is important to link the joints and the controller -->
+<robot name="six_arm" xmlns:xacro="http://www.ros.org/wiki/xacro">
+    <!-- <xacro:include filename="./large_base.xacro" /> -->
+    <xacro:include filename="$(find mybot_description)/urdf/large_base.xacro" />
+    <!-- Transmission is important to link the joints and the controller -->
+    <xacro:macro name="wheel_transmission" params="prefix">
         <transmission name="${prefix}_wheel_joint_trans">
             <type>transmission_interface/SimpleTransmission</type>
@@ -94,92 +15,41 @@
             </actuator>
         </transmission>
-    </xacro:macro>
-    <!-- Macro for robot 支撑轮 -->
-    <xacro:macro name="caster" params="prefix reflect">
-        <joint name="${prefix}_caster_joint" type="fixed">
-            <origin xyz="${reflect*caster_joint_x} 0 ${-(base_height/2 + caster_radius)}" rpy="0 0 0"/>
-            <parent link="base_link"/>
-            <child link="${prefix}_caster_link"/>
-        </joint>
-        <link name="${prefix}_caster_link">
-            <visual>
-                <origin xyz="0 0 0" rpy="0 0 0"/>
-                <geometry>
-                    <sphere radius="${caster_radius}" />
-                </geometry>
-                <material name="black" />
-            </visual>
-            <collision>
-                <origin xyz="0 0 0" rpy="0 0 0"/>
-                <geometry>
-                    <sphere radius="${caster_radius}" />
-                </geometry>
-            </collision>
-            <xacro:sphere_inertial_matrix m="${caster_mass}" r="${caster_radius}" />
-        </link>
-        <gazebo reference="${prefix}_caster_link">
-            <material>Gazebo/Black</material>
+        <gazebo reference="${prefix}_wheel_link">
+            <material>Gazebo/Gray</material>
+            <mu1>100000.0</mu1>
+            <mu2>100000.0</mu2>
         </gazebo>
     </xacro:macro>
-    <!-- 本体 -->
-    <xacro:macro name="base_gazebo">
-        <link name="base_footprint">
-            <visual>
-                <origin xyz="0 0 0" rpy="0 0 0" />
-                <geometry>
-                    <box size="0.001 0.001 0.001" />
-                </geometry>
-            </visual>
-        </link>
-        <gazebo reference="base_footprint">
-            <turnGravityOff>false</turnGravityOff>
-        </gazebo>
-        <joint name="base_footprint_joint" type="fixed">
-            <origin xyz="0 0 ${base_height/2 + caster_radius*2}" rpy="0 0 0" />
-            <parent link="base_footprint"/>
-            <child link="base_link" />
-        </joint>
-        <link name="base_link">
-            <visual>
-                <origin xyz=" 0 0 0" rpy="0 0 0" />
-                <geometry>
-                    <box size="${base_length} ${base_width} ${base_height}" />
-                </geometry>
-                <material name="yellow" />
-            </visual>
-            <collision>
-                <origin xyz=" 0 0 0" rpy="0 0 0" />
-                <geometry>
-                    <box size="${base_length} ${base_width} ${base_height}" />
-                </geometry>
-            </collision>
-            <xacro:box_inertial_matrix m="${base_mass}" l="${base_length}" w="${base_width}" h="${base_height}" />
-        </link>
-        <gazebo reference="base_link">
-            <material>Gazebo/Blue</material>
-        </gazebo>
-        <xacro:wheel prefix="left" reflect="1"/>
-        <xacro:wheel prefix="right" reflect="-1"/>
-        <xacro:caster prefix="back" reflect="-1"/>
-        <!-- controller -->
-        <gazebo>
-            <plugin name="differential_drive_controller" filename="libgazebo_ros_diff_drive.so">
-                <update_rate>30</update_rate>
-                <left_joint>left_wheel_joint</left_joint>
-                <right_joint>right_wheel_joint</right_joint>
-                <wheel_separation>${wheel_joint_y*2}</wheel_separation>
-                <wheel_diameter>${2*wheel_radius}</wheel_diameter>
-                <max_wheel_torque>10</max_wheel_torque>
-                <max_wheel_acceleration>1.0</max_wheel_acceleration>
-                <command_topic>cmd_vel</command_topic>
-                <publish_odom>true</publish_odom>
-                <publish_odom_tf>true</publish_odom_tf>
-                <publish_wheel_tf>true</publish_wheel_tf>
-                <odometry_topic>odom</odometry_topic>
-                <odometry_frame>odom</odometry_frame>
-                <robot_base_frame>base_footprint</robot_base_frame>
-                <odometry_source>1</odometry_source>
-            </plugin>
-        </gazebo>
-    </xacro:macro>
+    <!-- /////////////////////////////////   Gazebo   ////////////////////////////////////// -->
+    <gazebo reference="base_footprint">
+        <turnGravityOff>false</turnGravityOff>
+    </gazebo>
+    <gazebo reference="base_link">
+        <material>Gazebo/Blue</material>
+    </gazebo>
+    <gazebo reference="back_caster_link">
+        <material>Gazebo/Black</material>
+    </gazebo>
+    <xacro:wheel_transmission prefix="left" />
+    <xacro:wheel_transmission prefix="right" />
+    <!-- controller -->
+    <gazebo>
+        <plugin name="differential_drive_controller" filename="libgazebo_ros_diff_drive.so">
+            <update_rate>30</update_rate>
+            <left_joint>left_wheel_joint</left_joint>
+            <right_joint>right_wheel_joint</right_joint>
+            <wheel_separation>${wheel_joint_y*2}</wheel_separation>
+            <wheel_diameter>${2*wheel_radius}</wheel_diameter>
+            <max_wheel_torque>10</max_wheel_torque>
+            <max_wheel_acceleration>1.0</max_wheel_acceleration>
+            <command_topic>cmd_vel</command_topic>
+            <publish_odom>true</publish_odom>
+            <publish_odom_tf>true</publish_odom_tf>
+            <publish_wheel_tf>true</publish_wheel_tf>
+            <odometry_topic>odom</odometry_topic>
+            <odometry_frame>odom</odometry_frame>
+            <robot_base_frame>base_footprint</robot_base_frame>
+            <odometry_source>1</odometry_source>
+        </plugin>
+    </gazebo>
 </robot>

File: mybot_description/urdf/lidar_gazebo.xacro (robot description, xacro)
@@ -33,5 +33,4 @@
             <sensor type="ray" name="lidar">
                 <update_rate>20</update_rate>
-                <!-- <visualize>false</visualize> -->
                 <visualize>${gz_visualize}</visualize>
                 <ray>

File: mybot_description/urdf/originbot_with_rgbd_gazebo_arm.xacro (robot description, xacro)
@@ -4,8 +4,11 @@
     <xacro:include filename="$(find mybot_description)/urdf/large_base_gazebo.xacro" />
     <xacro:include filename="$(find mybot_description)/urdf/rgbd_gazebo.xacro" />
+    <xacro:include filename="$(find mybot_description)/urdf/camera_gazebo.xacro" />
     <xacro:include filename="$(find mybot_description)/urdf/lidar_gazebo.xacro" />
     <xacro:include filename="$(find mybot_description)/urdf/arm_gazebo.xacro" />
-    <!-- Base -->
-    <xacro:base_gazebo />
+    <!-- <xacro:include filename="./large_base_gazebo.xacro" />
+    <xacro:include filename="./rgbd_gazebo.xacro" />
+    <xacro:include filename="./lidar_gazebo.xacro" />
+    <xacro:include filename="./arm_gazebo.xacro" /> -->
     <!-- rgbd -->
     <xacro:property name="rgbd_offset_x" value="${base_length/2+0.02}" />
@@ -13,9 +16,19 @@
     <xacro:property name="rgbd_offset_z" value="0.02" />
     <joint name="rgbd_joint" type="fixed">
-        <origin xyz="${rgbd_offset_x} ${rgbd_offset_y} ${rgbd_offset_z}" rpy="0 0 0" />
+        <origin xyz="${-rgbd_offset_x} ${rgbd_offset_y} ${rgbd_offset_z}" rpy="0 ${-M_PI/2} 0" />
+        <parent link="grasping_frame" />
+        <child link="camera_rgbd_link" />
+    </joint>
+    <xacro:rgbd_camera prefix="camera_rgbd" />
+    <!-- Camera -->
+    <xacro:property name="camera_offset_x" value="${base_length/2+0.02}" />
+    <xacro:property name="camera_offset_y" value="0" />
+    <xacro:property name="camera_offset_z" value="-0.01" />
+    <joint name="camera_joint" type="fixed">
+        <origin xyz="${camera_offset_x} ${camera_offset_y} ${camera_offset_z}" rpy="0 0 0" />
         <parent link="base_link" />
         <child link="camera_link" />
     </joint>
-    <xacro:rgbd_camera prefix="camera" />
+    <xacro:mipi_camera prefix="camera" />
     <!-- Lidar -->
     <xacro:property name="lidar_offset_x" value="0" />
@@ -29,5 +42,7 @@
         <child link="laser_link" />
     </joint>
-    <xacro:lidar prefix="laser" gz_visualize="false" range_min="${robot_radius + safety_margin}" />
+    <xacro:lidar prefix="laser" gz_visualize="false" range_min="0.5" />
+    <!-- <xacro:lidar prefix="laser" gz_visualize="false" range_min="${robot_radius +
+    safety_margin}" /> -->
     <!-- arm -->
     <xacro:property name="arm_offset_x" value="0.0" />
@@ -35,5 +50,5 @@
     <xacro:property name="arm_offset_z" value="${base_height/2+0.01}" />
     <joint name="connect_joint" type="fixed">
-        <origin xyz="${arm_offset_x} ${arm_offset_y} ${arm_offset_z}" rpy="0 0 0" />
+        <origin xyz="${arm_offset_x} ${arm_offset_y} ${arm_offset_z}" rpy=" 0 0 0" />
         <parent link="base_link" />
         <child link="arm_base_link" />

File: mybot_description/urdf/rgbd_gazebo.xacro (robot description, xacro)
@@ -43,10 +43,10 @@
                 <plugin name="${prefix}_controller" filename="libgazebo_ros_camera.so">
                     <ros>
-                        <!-- <namespace>${prefix}</namespace> -->
-                        <remapping>${prefix}/image_raw:=camera/image_raw</remapping>
-                        <remapping>${prefix}/image_depth:=depth/image_raw</remapping>
-                        <remapping>${prefix}/camera_info:=camera/camera_info</remapping>
-                        <remapping>${prefix}/camera_info_depth:=depth/camera_info</remapping>
-                        <remapping>${prefix}/points:=depth/points</remapping>
+                        <namespace>${prefix}</namespace>
+                        <!-- <remapping>${prefix}/image_raw:=camera/image_raw</remapping> -->
+                        <!-- <remapping>${prefix}/image_depth:=depth/image_raw</remapping> -->
+                        <!-- <remapping>${prefix}/camera_info:=camera/camera_info</remapping> -->
+                        <!-- <remapping>${prefix}/camera_info_depth:=depth/camera_info</remapping> -->
+                        <!-- <remapping>${prefix}/points:=depth/points</remapping> -->
                     </ros>
                     <camera_name>${prefix}</camera_name>
