Commit message: 发布第一版

File: mybot_description/urdf/arm.xacro (robot description, xacro)
@@ -31,5 +31,5 @@
     <xacro:property name="link5_len" value="0.06" />
     <!-- link6 -->
-    <xacro:property name="link6_rad" value="0.04" />
+    <xacro:property name="link6_rad" value="0.05" />
     <xacro:property name="link6_len" value="0.02" />
     <!-- 夹爪 长宽高-->
@@ -38,4 +38,7 @@
     <xacro:property name="gripper_w" value="0.01" />
     <xacro:property name="gripper_h" value="0.02" />
+    <!-- 夹爪安装距离参数0~1 -->
+    <xacro:property name="gripper_offset" value="0.75" />
+    <xacro:property name="gripper_offset_h" value="0.002" />
     <!-- 底座长宽高 -->
     <!-- base -->
@@ -246,44 +249,36 @@
     </joint>
     <!-- 夹爪 -->
-    <link name="gripper_finger_link1">
-        <visual>
-            <geometry>
-                <box size="${gripper_l} ${gripper_w} ${gripper_h}" />
-            </geometry>
-            <material name="White" />
-        </visual>
-        <collision>
-            <geometry>
-                <box size="${gripper_l} ${gripper_w} ${gripper_h}" />
-            </geometry>
-        </collision>
-        <xacro:inertial_matrix m="0.01" />
-    </link>
+    <xacro:macro name="gripper_finger_link" params="num">
+        <link name="gripper_finger_link${num}">
+            <visual>
+                <geometry>
+                    <box size="${gripper_l} ${gripper_w} ${gripper_h}" />
+                </geometry>
+                <material name="White" />
+            </visual>
+            <collision>
+                <geometry>
+                    <box size="${gripper_l} ${gripper_w} ${gripper_h}" />
+                </geometry>
+            </collision>
+            <xacro:inertial_matrix m="0.01" />
+        </link>
+    </xacro:macro>
+    <xacro:gripper_finger_link num="1" />
+    <xacro:gripper_finger_link num="2" />
     <joint name="finger_joint1" type="prismatic">
         <parent link="link6" />
         <child link="gripper_finger_link1" />
-        <origin xyz="0 -${link6_rad *0.6} ${gripper_h}" rpy="0 ${M_PI/2} 0" />
+        <origin xyz="0 -${link6_rad *gripper_offset} ${gripper_h*2+gripper_offset_h}"
+            rpy="0 ${M_PI/2} 0" />
         <axis xyz="0 1 0" />
-        <limit effort="100" lower="0" upper="${link6_rad}" velocity="1.0" />
+        <limit effort="100" lower="0" upper="${link6_rad+gripper_w}" velocity="1.0" />
         <dynamics damping="50" friction="1" />
     </joint>
-    <link name="gripper_finger_link2">
-        <visual>
-            <geometry>
-                <box size="${gripper_l} ${gripper_w} ${gripper_h}" />
-            </geometry>
-            <material name="White" />
-        </visual>
-        <collision>
-            <geometry>
-                <box size="${gripper_l} ${gripper_w} ${gripper_h}" />
-            </geometry>
-        </collision>
-        <xacro:inertial_matrix m="0.01" />
-    </link>
     <joint name="finger_joint2" type="fixed">
         <parent link="link6" />
         <child link="gripper_finger_link2" />
-        <origin xyz="0 ${link6_rad *0.75} ${gripper_h}" rpy="0 ${M_PI/2} 0" />
+        <origin xyz="0 ${link6_rad *gripper_offset} ${gripper_h*2+gripper_offset_h}"
+            rpy="0 ${M_PI/2} 0" />
     </joint>
     <!-- Grasping frame -->

File: mybot_description/urdf/large_base_gazebo.xacro (robot description, xacro)
@@ -1,5 +1,4 @@
 <?xml version="1.0"?>
 <robot name="six_arm" xmlns:xacro="http://www.ros.org/wiki/xacro">
-    <!-- <xacro:include filename="./large_base.xacro" /> -->
     <xacro:include filename="$(find mybot_description)/urdf/large_base.xacro" />
     <!-- Transmission is important to link the joints and the controller -->

File: mybot_description/urdf/originbot_with_rgbd_gazebo_arm.xacro (robot description, xacro)
@@ -7,12 +7,8 @@
     <xacro:include filename="$(find mybot_description)/urdf/lidar_gazebo.xacro" />
     <xacro:include filename="$(find mybot_description)/urdf/arm_gazebo.xacro" />
-    <!-- <xacro:include filename="./large_base_gazebo.xacro" />
-    <xacro:include filename="./rgbd_gazebo.xacro" />
-    <xacro:include filename="./lidar_gazebo.xacro" />
-    <xacro:include filename="./arm_gazebo.xacro" /> -->
     <!-- rgbd -->
-    <xacro:property name="rgbd_offset_x" value="${base_length/2+0.02}" />
+    <xacro:property name="rgbd_offset_x" value="0.06" />
     <xacro:property name="rgbd_offset_y" value="0" />
-    <xacro:property name="rgbd_offset_z" value="0.02" />
+    <xacro:property name="rgbd_offset_z" value="-0.03" />
     <joint name="rgbd_joint" type="fixed">
         <origin xyz="${-rgbd_offset_x} ${rgbd_offset_y} ${rgbd_offset_z}" rpy="0 ${-M_PI/2} 0" />

Commit message: 模型微调

File: mybot_description/urdf/arm.xacro (robot description, xacro)
@@ -219,5 +219,5 @@
         <origin xyz="0 0 ${link4_len}" rpy="0 0 0" />
         <axis xyz="0 -1 0" />
-        <limit effort="300" velocity="1.0" lower="-2.35" upper="2.35" />
+        <limit effort="300" velocity="1.0" lower="-2.04" upper="2.04" />
         <joint_properties damping="50" friction="1" />
     </joint>

File: mybot_description/urdf/large_base.xacro (robot description, xacro)
@@ -5,5 +5,5 @@
     <!-- PROPERTY LIST -->
     <xacro:property name="M_PI" value="3.1415926" />
-    <xacro:property name="base_mass" value="2" />
+    <xacro:property name="base_mass" value="4" />
     <xacro:property name="base_width" value="0.320" />
     <xacro:property name="base_length" value="0.320" />
@@ -13,11 +13,17 @@
     <xacro:property name="wheel_radius" value="0.065" />
     <xacro:property name="wheel_length" value="0.050" />
-    <xacro:property name="wheel_joint_x" value="0.14" />
-    <xacro:property name="wheel_joint_y" value="0.38" />
-    <xacro:property name="wheel_joint_z" value="0.035" />
+    <!-- base_length/2 = 0.16; x偏移-0.02-->
+    <xacro:property name="wheel_joint_x" value="${base_length/2 - 0.02}" />
+    <!-- (base_width+wheel_length)/2 -->
+    <xacro:property name="wheel_joint_y" value="${(base_width+wheel_length)/2}" />
+    <!-- base_height/2 = 0.05;向上偏移一点（-0.015）  -->
+    <xacro:property name="wheel_joint_z" value="${base_height/2 - 0.015}" />
     <!-- 支撑轮 -->
     <xacro:property name="caster_mass" value="0.4" />
-    <xacro:property name="caster_radius" value="0.0267" />
-    <xacro:property name="caster_joint_x" value="0.14" />
+    <!-- 计算中心到地面高度，再减去底盘得到底盘到地面高度:
+    wheel_joint_z + wheel_radius  - base_height/2; -->
+    <xacro:property name="caster_radius" value="${(wheel_joint_z + wheel_radius - base_height/2)/2}" />
+    <!-- 与前轮对称 -->
+    <xacro:property name="caster_joint_x" value="${wheel_joint_x}" />
     <material name="yellow">
         <color rgba="1 0.4 0 1" />
@@ -57,5 +63,5 @@
     <xacro:macro name="wheel" params="prefix reflect">
         <joint name="${prefix}_wheel_joint" type="continuous">
-            <origin xyz="${wheel_joint_x} ${reflect*(base_width+wheel_length)/2} ${-wheel_joint_z}"
+            <origin xyz="${wheel_joint_x} ${reflect*wheel_joint_y} ${-wheel_joint_z}"
                 rpy="0 0 0" />
             <parent link="base_link" />
@@ -127,10 +133,10 @@
             <material name="yellow" />
         </visual>
-        <collision>
+        <!-- <collision>
             <origin xyz=" 0 0 0" rpy="0 0 0" />
             <geometry>
                 <box size="${base_length} ${base_width} ${base_height}" />
             </geometry>
-        </collision>
+        </collision> -->
         <xacro:box_inertial_matrix m="${base_mass}" l="${base_length}" w="${base_width}"
             h="${base_height}" />

File: mybot_description/urdf/lidar_gazebo.xacro (robot description, xacro)
@@ -32,5 +32,5 @@
         <gazebo reference="${prefix}_link">
             <sensor type="ray" name="lidar">
-                <update_rate>20</update_rate>
+                <update_rate>10</update_rate>
                 <visualize>${gz_visualize}</visualize>
                 <ray>
@@ -38,7 +38,7 @@
                         <horizontal>
                             <samples>360</samples>
-                            <resolution>1</resolution>
-                            <min_angle>-3.14</min_angle>
-                            <max_angle>3.14</max_angle>
+                            <resolution>0.5</resolution>
+                            <min_angle>-3.14159</min_angle>
+                            <max_angle>3.14159</max_angle>
                         </horizontal>
                     </scan>
@@ -51,5 +51,5 @@
                         <type>gaussian</type>
                         <mean>0.0</mean>
-                        <stddev>0.01</stddev>
+                        <stddev>0.005</stddev>
                     </noise>
                 </ray>

Commit message: 重构mybot描述文件，移除冗余惯性矩阵宏，优化arm和large_base的URDF配置，添加Gazebo启动脚本及MoveIt配置

File: mybot_description/urdf/arm.xacro (robot description, xacro)
@@ -53,29 +53,4 @@
         </inertial>
     </xacro:macro>
-    <!-- Macro for inertia matrix -->
-    <xacro:macro name="sphere_inertial_matrix" params="m r">
-        <inertial>
-            <mass value="${m}" />
-            <inertia ixx="${2*m*r*r/5}" ixy="0" ixz="0"
-                iyy="${2*m*r*r/5}" iyz="0"
-                izz="${2*m*r*r/5}" />
-        </inertial>
-    </xacro:macro>
-    <xacro:macro name="cylinder_inertial_matrix" params="m r h">
-        <inertial>
-            <mass value="${m}" />
-            <inertia ixx="${m*(3*r*r+h*h)/12}" ixy="0" ixz="0"
-                iyy="${m*(3*r*r+h*h)/12}" iyz="0"
-                izz="${m*r*r/2}" />
-        </inertial>
-    </xacro:macro>
-    <xacro:macro name="box_inertial_matrix" params="m l w h">
-        <inertial>
-            <mass value="${m}" />
-            <inertia ixx="${m*(h*h + l*l)/12}" ixy="0" ixz="0"
-                iyy="${m*(w*w + l*l)/12}" iyz="0"
-                izz="${m*(w*w + h*h)/12}" />
-        </inertial>
-    </xacro:macro>
     <!-- 底座 -->
     <link name="arm_base_link">
@@ -92,5 +67,5 @@
             </geometry>
         </collision>
-        <xacro:inertial_matrix m="1" />
+        <xacro:inertial_matrix m="0.1" />
     </link>
     <!-- joint1 -->

File: mybot_description/urdf/large_base.xacro (robot description, xacro)
@@ -36,27 +36,13 @@
     </material>
     <!-- Macro for inertia matrix -->
-    <!-- 球面惯性矩阵 -->
-    <xacro:macro name="sphere_inertial_matrix" params="m r">
-        <inertial>
-            <mass value="${m}" />
-            <inertia ixx="${2*m*r*r/5}" ixy="0" ixz="0" iyy="${2*m*r*r/5}" iyz="0"
-                izz="${2*m*r*r/5}" />
-        </inertial>
-    </xacro:macro>
-    <!-- 圆柱惯性矩阵 -->
-    <xacro:macro name="cylinder_inertial_matrix" params="m r h">
-        <inertial>
-            <mass value="${m}" />
-            <inertia ixx="${m*(3*r*r+h*h)/12}" ixy="0" ixz="0" iyy="${m*(3*r*r+h*h)/12}" iyz="0"
-                izz="${m*r*r/2}" />
-        </inertial>
-    </xacro:macro>
-    <!-- 方块惯性矩阵 -->
-    <xacro:macro name="box_inertial_matrix" params="m l w h">
-        <inertial>
-            <mass value="${m}" />
-            <inertia ixx="${m*(h*h + l*l)/12}" ixy="0" ixz="0" iyy="${m*(w*w + l*l)/12}" iyz="0"
-                izz="${m*(w*w + h*h)/12}" />
-        </inertial>
+    <!-- 正立方体（边长 s，质量 m）惯性矩阵模板 -->
+    <xacro:macro name="inertial_matrix" params="m s">
+    <xacro:property name="i" value="${m*s*s/6}" />
+    <inertial>
+        <mass value="${m}" />
+        <inertia  ixx="${i}" ixy="0" ixz="0"
+                iyy="${i}" iyz="0"
+                izz="${i}" />
+    </inertial>
     </xacro:macro>
     <!-- Macro for robot 轮子 -->
@@ -83,6 +69,5 @@
                 </geometry>
             </collision>
-            <xacro:cylinder_inertial_matrix m="${wheel_mass}" r="${wheel_radius}"
-                h="${wheel_length}" />
+            <xacro:inertial_matrix m="${wheel_mass}" s="${caster_radius}" />
         </link>
     </xacro:macro>
@@ -109,5 +94,5 @@
                 </geometry>
             </collision>
-            <xacro:sphere_inertial_matrix m="${caster_mass}" r="${caster_radius}" />
+            <!-- <xacro:inertial_matrix m="${caster_mass}" s="${caster_radius}" /> -->
         </link>
     </xacro:macro>
@@ -136,9 +121,8 @@
             <origin xyz=" 0 0 0" rpy="0 0 0" />
             <geometry>
-                <box size="${base_length} ${base_width} ${base_height}" />
+                <box size="${base_length*0.1} ${base_width*0.1} ${base_height*0.1}" />
             </geometry>
         </collision> -->
-        <xacro:box_inertial_matrix m="${base_mass}" l="${base_length}" w="${base_width}"
-            h="${base_height}" />
+        <xacro:inertial_matrix m="${base_mass}" s="${base_height*0.5}" />
     </link>
     <xacro:wheel prefix="left" reflect="1" />

File: mybot_description/urdf/originbot_with_rgbd_gazebo_arm.xacro (robot description, xacro)
@@ -2,9 +2,10 @@
 <robot name="six_arm"
     xmlns:xacro="http://www.ros.org/wiki/xacro">
-    <xacro:include filename="$(find mybot_description)/urdf/large_base_gazebo.xacro" />
+    <!-- <xacro:include filename="$(find mybot_description)/urdf/large_base_gazebo.xacro" /> -->
+    <!-- <xacro:include filename="$(find mybot_description)/urdf/arm_gazebo.xacro" /> -->
+    <xacro:include filename="$(find mybot_description)/urdf/originbot_with_arm_gazebo.xacro" />
     <xacro:include filename="$(find mybot_description)/urdf/rgbd_gazebo.xacro" />
     <xacro:include filename="$(find mybot_description)/urdf/camera_gazebo.xacro" />
     <xacro:include filename="$(find mybot_description)/urdf/lidar_gazebo.xacro" />
-    <xacro:include filename="$(find mybot_description)/urdf/arm_gazebo.xacro" />
     <!-- rgbd -->
     <xacro:property name="rgbd_offset_x" value="0.06" />
@@ -38,15 +39,5 @@
         <child link="laser_link" />
     </joint>
-    <xacro:lidar prefix="laser" gz_visualize="false" range_min="0.5" />
-    <!-- <xacro:lidar prefix="laser" gz_visualize="false" range_min="${robot_radius +
-    safety_margin}" /> -->
-    <!-- arm -->
-    <xacro:property name="arm_offset_x" value="0.0" />
-    <xacro:property name="arm_offset_y" value="0" />
-    <xacro:property name="arm_offset_z" value="${base_height/2+0.01}" />
-    <joint name="connect_joint" type="fixed">
-        <origin xyz="${arm_offset_x} ${arm_offset_y} ${arm_offset_z}" rpy=" 0 0 0" />
-        <parent link="base_link" />
-        <child link="arm_base_link" />
-    </joint>
+    <!-- <xacro:lidar prefix="laser" gz_visualize="false" range_min="0.5" /> -->
+    <xacro:lidar prefix="laser" gz_visualize="true" range_min="${robot_radius + safety_margin}" />
 </robot>

File: mybot_description/urdf/rgbd_gazebo.xacro (robot description, xacro)
@@ -12,9 +12,4 @@
                 </geometry>
             </visual>
-            <collision>
-                <geometry>
-                    <box size="0.07 0.3 0.09" />
-                </geometry>
-            </collision>
         </link>
         <joint name="${prefix}_optical_joint" type="fixed">
