Commit message: 添加imu传感器，调整参数，更健康的参数，不会乱飞

File: mybot_description/urdf/arm.xacro (robot description, xacro)
@@ -14,4 +14,5 @@
     <!-- 常量 -->
     <xacro:property name="M_PI" value="3.1415926" />
+    <xacro:property name="P" value="600.0" />
     <!-- 连杆半径和长度 -->
     <!-- link1 -->
@@ -47,10 +48,26 @@
     <xacro:property name="base_h" value="0.04" />
     <!-- 惯性矩阵 -->
-    <xacro:macro name="inertial_matrix" params="m">
+    <!-- <xacro:macro name="inertial_matrix" params="m">
         <inertial>
             <mass value="${m}" />
             <inertia ixx="0.0001" ixy="0" ixz="0" iyy="0.0001" iyz="0" izz="0.0001" />
         </inertial>
+    </xacro:macro> -->
+    <xacro:macro name="box_i" params="w h d">
+        <inertial>
+        <origin xyz="0 0 0" rpy="${pi/2} 0 ${pi/2}"/>
+        <xacro:property name="m" value="${w*h*d*P}" />
+        <mass value="${m}"/>
+        <inertia ixx="${(m/12) * (h*h + d*d)}" ixy="0.0" ixz="0.0" iyy="${(m/12) * (w*w + d*d)}" iyz="0.0" izz="${(m/12) * (w*w + h*h)}"/>
+        </inertial>
     </xacro:macro>
+    <xacro:macro name="cylinder_i" params="r h">
+        <inertial>
+        <origin xyz="0 0 0" rpy="${pi/2} 0 0" />
+        <xacro:property name="m" value="${(pi*r*r*h*P)}" />
+        <mass value="${m}"/>
+        <inertia ixx="${(m/12) * (3*r*r + h*h)}" ixy = "0" ixz = "0" iyy="${(m/12) * (3*r*r + h*h)}" iyz = "0" izz="${(m/2) * (r*r)}"/>
+        </inertial>
+  </xacro:macro>
     <!-- 底座 -->
     <link name="arm_base_link">
@@ -67,5 +84,6 @@
             </geometry>
         </collision>
-        <xacro:inertial_matrix m="0.1" />
+        <!-- <xacro:inertial_matrix m="0.1" /> -->
+        <xacro:box_i w="${base_w}" h="${base_h}" d="${base_l}" />
     </link>
     <!-- joint1 -->
@@ -91,5 +109,6 @@
             </geometry>
         </collision>
-        <xacro:inertial_matrix m="0.1" />
+        <!-- <xacro:inertial_matrix m="0.1" /> -->
+        <xacro:cylinder_i r="${link1_rad}" h="${link1_len}" />
     </link>
     <!-- link2 -->
@@ -108,5 +127,6 @@
             </geometry>
         </collision>
-        <xacro:inertial_matrix m="0.1" />
+        <!-- <xacro:inertial_matrix m="0.1" /> -->
+        <xacro:cylinder_i r="${link2_rad}" h="${link2_len}" />
     </link>
     <!-- joint2 -->
@@ -134,5 +154,6 @@
             </geometry>
         </collision>
-        <xacro:inertial_matrix m="0.1" />
+        <!-- <xacro:inertial_matrix m="0.1" /> -->
+        <xacro:cylinder_i r="${link3_rad}" h="${link3_len}" />
     </link>
     <!-- joint3 -->
@@ -160,5 +181,6 @@
             </geometry>
         </collision>
-        <xacro:inertial_matrix m="0.1" />
+        <!-- <xacro:inertial_matrix m="0.1" /> -->
+        <xacro:cylinder_i r="${link4_rad}" h="${link4_len}" />
     </link>
     <!-- joint4 -->
@@ -186,5 +208,6 @@
             </geometry>
         </collision>
-        <xacro:inertial_matrix m="0.1" />
+        <!-- <xacro:inertial_matrix m="0.1" /> -->
+        <xacro:cylinder_i r="${link5_rad}" h="${link5_len}" />
     </link>
     <!-- joint5 -->
@@ -212,5 +235,6 @@
             </geometry>
         </collision>
-        <xacro:inertial_matrix m="0.1" />
+        <!-- <xacro:inertial_matrix m="0.1" /> -->
+        <xacro:cylinder_i r="${link6_rad}" h="${link6_len}" />
     </link>
     <!-- joint6 -->
@@ -237,5 +261,6 @@
                 </geometry>
             </collision>
-            <xacro:inertial_matrix m="0.01" />
+            <!-- <xacro:inertial_matrix m="0.01" /> -->
+            <xacro:box_i d="${gripper_l}" w="${gripper_w}" h="${gripper_h}" />
         </link>
     </xacro:macro>

File: mybot_description/urdf/large_base.xacro (robot description, xacro)
@@ -5,17 +5,17 @@
     <!-- PROPERTY LIST -->
     <xacro:property name="M_PI" value="3.1415926" />
-    <xacro:property name="base_mass" value="4" />
-    <xacro:property name="base_width" value="0.320" />
-    <xacro:property name="base_length" value="0.320" />
+    <xacro:property name="base_mass" value="6" />
+    <xacro:property name="base_width" value="0.480" />
+    <xacro:property name="base_length" value="0.480" />
     <xacro:property name="base_height" value="0.1" />
     <!-- 轮子 -->
-    <xacro:property name="wheel_mass" value="0.4" />
+    <xacro:property name="wheel_mass" value="1" />
     <xacro:property name="wheel_radius" value="0.065" />
     <xacro:property name="wheel_length" value="0.050" />
     <!-- base_length/2 = 0.16; x偏移-0.02-->
     <xacro:property name="wheel_joint_x" value="${base_length/2 - 0.02}" />
-    <!-- (base_width+wheel_length)/2 -->
+    <!-- (base_width+wheel_length)/2 轮距 -->
     <xacro:property name="wheel_joint_y" value="${(base_width+wheel_length)/2}" />
-    <!-- base_height/2 = 0.05;向上偏移一点（-0.015）  -->
+    <!-- base_height/2 = 0.05;向上偏移一点（-0.015） -->
     <xacro:property name="wheel_joint_z" value="${base_height/2 - 0.015}" />
     <!-- 支撑轮 -->
@@ -26,4 +26,5 @@
     <!-- 与前轮对称 -->
     <xacro:property name="caster_joint_x" value="${wheel_joint_x}" />
+    <xacro:property name="caster_joint_y" value="${base_width/2-caster_radius}" />
     <material name="yellow">
         <color rgba="1 0.4 0 1" />
@@ -36,5 +37,4 @@
     </material>
     <!-- Macro for inertia matrix -->
-    <!-- 正立方体（边长 s，质量 m）惯性矩阵模板 -->
     <xacro:macro name="inertial_matrix" params="m s">
     <xacro:property name="i" value="${m*s*s/6}" />
@@ -44,4 +44,18 @@
                 iyy="${i}" iyz="0"
                 izz="${i}" />
+    </inertial>
+    </xacro:macro>
+    <xacro:macro name="box_inertia" params="m w h d">
+    <inertial>
+      <origin xyz="0 0 0" rpy="${pi/2} 0 ${pi/2}"/>
+      <mass value="${m}"/>
+      <inertia ixx="${(m/12) * (h*h + d*d)}" ixy="0.0" ixz="0.0" iyy="${(m/12) * (w*w + d*d)}" iyz="0.0" izz="${(m/12) * (w*w + h*h)}"/>
+    </inertial>
+    </xacro:macro>
+    <xacro:macro name="cylinder_inertia" params="m r h">
+    <inertial>
+      <origin xyz="0 0 0" rpy="${pi/2} 0 0" />
+      <mass value="${m}"/>
+      <inertia ixx="${(m/12) * (3*r*r + h*h)}" ixy = "0" ixz = "0" iyy="${(m/12) * (3*r*r + h*h)}" iyz = "0" izz="${(m/2) * (r*r)}"/>
     </inertial>
     </xacro:macro>
@@ -70,4 +84,5 @@
             </collision>
             <xacro:inertial_matrix m="${wheel_mass}" s="${caster_radius}" />
+            <!-- <xacro:cylinder_inertia m="${wheel_mass}" r="${wheel_radius}" h="${wheel_length}" /> -->
         </link>
     </xacro:macro>
@@ -75,5 +90,5 @@
     <xacro:macro name="caster" params="prefix reflect">
         <joint name="${prefix}_caster_joint" type="fixed">
-            <origin xyz="${reflect*caster_joint_x} 0 ${-(base_height/2 + caster_radius)}"
+            <origin xyz="${-1*caster_joint_x} ${reflect*caster_joint_y} ${-(base_height/2 + caster_radius)}"
                 rpy="0 0 0" />
             <parent link="base_link" />
@@ -94,5 +109,5 @@
                 </geometry>
             </collision>
-            <!-- <xacro:inertial_matrix m="${caster_mass}" s="${caster_radius}" /> -->
+            <xacro:inertial_matrix m="${caster_mass}" s="${caster_radius}" />
         </link>
     </xacro:macro>
@@ -124,8 +139,9 @@
             </geometry>
         </collision> -->
-        <xacro:inertial_matrix m="${base_mass}" s="${base_height*0.5}" />
+        <xacro:box_inertia m="${base_mass}" w="${base_width}" h="${base_height}" d="${base_length}" />
     </link>
     <xacro:wheel prefix="left" reflect="1" />
     <xacro:wheel prefix="right" reflect="-1" />
-    <xacro:caster prefix="back" reflect="-1" />
+    <xacro:caster prefix="backr" reflect="-1" />
+    <xacro:caster prefix="backl" reflect="1" />
 </robot>

File: mybot_description/urdf/originbot_with_arm_gazebo.xacro (robot description, xacro)
@@ -68,5 +68,5 @@
     <gazebo>
         <plugin name="gazebo_ros2_control" filename="libgazebo_ros2_control.so">
-            <parameters>$(find mybotp)/config/ros2_controllers.yaml</parameters>
+            <parameters>$(find mybot)/config/ros2_controllers.yaml</parameters>
             <robot_param_node>robot_state_publisher</robot_param_node>
         </plugin>
@@ -79,5 +79,8 @@
         <material>Gazebo/Blue</material>
     </gazebo>
-    <gazebo reference="back_caster_link">
+    <gazebo reference="backl_caster_link">
+        <material>Gazebo/Black</material>
+    </gazebo>
+    <gazebo reference="backr_caster_link">
         <material>Gazebo/Black</material>
     </gazebo>
@@ -103,11 +106,18 @@
     <gazebo>
         <plugin name="differential_drive_controller" filename="libgazebo_ros_diff_drive.so">
+            <!-- <ros>
+                <namespace>/demo</namespace>
+            </ros> -->
             <update_rate>30</update_rate>
+            <!-- wheels -->
             <left_joint>left_wheel_joint</left_joint>
             <right_joint>right_wheel_joint</right_joint>
+            <!-- kinematics -->
             <wheel_separation>${wheel_joint_y*2}</wheel_separation>
             <wheel_diameter>${2*wheel_radius}</wheel_diameter>
-            <max_wheel_torque>10</max_wheel_torque>
+            <!-- limits -->
+            <max_wheel_torque>20</max_wheel_torque>
             <max_wheel_acceleration>1.0</max_wheel_acceleration>
+            <!-- output -->
             <command_topic>cmd_vel</command_topic>
             <publish_odom>true</publish_odom>
@@ -117,5 +127,4 @@
             <odometry_frame>odom</odometry_frame>
             <robot_base_frame>base_footprint</robot_base_frame>
-            <odometry_source>1</odometry_source>
         </plugin>
     </gazebo>

File: mybot_description/urdf/originbot_with_rgbd_gazebo_arm.xacro (robot description, xacro)
@@ -8,4 +8,5 @@
     <xacro:include filename="$(find mybot_description)/urdf/camera_gazebo.xacro" />
     <xacro:include filename="$(find mybot_description)/urdf/lidar_gazebo.xacro" />
+    <xacro:include filename="$(find mybot_description)/urdf/imu_gazebo.xacro" />
     <!-- rgbd -->
     <xacro:property name="rgbd_offset_x" value="0.06" />
@@ -41,3 +42,5 @@
     <!-- <xacro:lidar prefix="laser" gz_visualize="false" range_min="0.5" /> -->
     <xacro:lidar prefix="laser" gz_visualize="true" range_min="${robot_radius + safety_margin}" />
+    <!-- IMU -->
+    <xacro:imu_sensor parent_link="base_link" />
 </robot>

File: mybot_description/urdf/rgbd_gazebo.xacro (robot description, xacro)
@@ -12,4 +12,8 @@
                 </geometry>
             </visual>
+            <inertial>
+                <mass value="0.1" />
+                <inertia ixx="0.0001" ixy="0" ixz="0" iyy="0.0001" iyz="0" izz="0.0001" />
+            </inertial>
         </link>
         <joint name="${prefix}_optical_joint" type="fixed">
