Commit message: 替换旧的功能包，添加ekf_filter_node

File: mybot/config/six_arm.ros2_control.xacro (robot description, xacro)
@@ -1,64 +1,62 @@
 <?xml version="1.0"?>
 <robot xmlns:xacro="http://www.ros.org/wiki/xacro">
-  <xacro:macro name="six_arm_ros2_control" params="name initial_positions_file">
-    <xacro:property name="initial_positions"
-      value="${xacro.load_yaml(initial_positions_file)['initial_positions']}" />
-    <!-- <xacro:property name="initial_positions"
-    value="${load_yaml(initial_positions_file)['initial_positions']}"/> -->
-    <ros2_control name="${name}" type="system">
-      <hardware>
-        <!-- By default, set up controllers for simulation. This won't work on real hardware -->
-        <plugin>mock_components/GenericSystem</plugin>
-      </hardware>
-      <joint name="joint1">
-        <command_interface name="position" />
-        <state_interface name="position">
-          <param name="initial_value">${initial_positions['joint1']}</param>
-        </state_interface>
-        <state_interface name="velocity" />
-      </joint>
-      <joint name="joint2">
-        <command_interface name="position" />
-        <state_interface name="position">
-          <param name="initial_value">${initial_positions['joint2']}</param>
-        </state_interface>
-        <state_interface name="velocity" />
-      </joint>
-      <joint name="joint3">
-        <command_interface name="position" />
-        <state_interface name="position">
-          <param name="initial_value">${initial_positions['joint3']}</param>
-        </state_interface>
-        <state_interface name="velocity" />
-      </joint>
-      <joint name="joint4">
-        <command_interface name="position" />
-        <state_interface name="position">
-          <param name="initial_value">${initial_positions['joint4']}</param>
-        </state_interface>
-        <state_interface name="velocity" />
-      </joint>
-      <joint name="joint5">
-        <command_interface name="position" />
-        <state_interface name="position">
-          <param name="initial_value">${initial_positions['joint5']}</param>
-        </state_interface>
-        <state_interface name="velocity" />
-      </joint>
-      <joint name="joint6">
-        <command_interface name="position" />
-        <state_interface name="position">
-          <param name="initial_value">${initial_positions['joint6']}</param>
-        </state_interface>
-        <state_interface name="velocity" />
-      </joint>
-      <joint name="finger_joint1">
-        <command_interface name="position" />
-        <state_interface name="position">
-          <param name="initial_value">${initial_positions['finger_joint1']}</param>
-        </state_interface>
-        <state_interface name="velocity" />
-      </joint>
-    </ros2_control>
-  </xacro:macro>
+    <xacro:macro name="six_arm_ros2_control" params="name initial_positions_file">
+        <xacro:property name="initial_positions" value="${xacro.load_yaml(initial_positions_file)['initial_positions']}"/>
+        <!-- <xacro:property name="initial_positions" value="${load_yaml(initial_positions_file)['initial_positions']}"/> -->
+        <ros2_control name="${name}" type="system">
+            <hardware>
+                <!-- By default, set up controllers for simulation. This won't work on real hardware -->
+                <plugin>mock_components/GenericSystem</plugin>
+            </hardware>
+            <joint name="joint1">
+                <command_interface name="position"/>
+                <state_interface name="position">
+                  <param name="initial_value">${initial_positions['joint1']}</param>
+                </state_interface>
+                <state_interface name="velocity"/>
+            </joint>
+            <joint name="joint2">
+                <command_interface name="position"/>
+                <state_interface name="position">
+                  <param name="initial_value">${initial_positions['joint2']}</param>
+                </state_interface>
+                <state_interface name="velocity"/>
+            </joint>
+            <joint name="joint3">
+                <command_interface name="position"/>
+                <state_interface name="position">
+                  <param name="initial_value">${initial_positions['joint3']}</param>
+                </state_interface>
+                <state_interface name="velocity"/>
+            </joint>
+            <joint name="joint4">
+                <command_interface name="position"/>
+                <state_interface name="position">
+                  <param name="initial_value">${initial_positions['joint4']}</param>
+                </state_interface>
+                <state_interface name="velocity"/>
+            </joint>
+            <joint name="joint5">
+                <command_interface name="position"/>
+                <state_interface name="position">
+                  <param name="initial_value">${initial_positions['joint5']}</param>
+                </state_interface>
+                <state_interface name="velocity"/>
+            </joint>
+            <joint name="joint6">
+                <command_interface name="position"/>
+                <state_interface name="position">
+                  <param name="initial_value">${initial_positions['joint6']}</param>
+                </state_interface>
+                <state_interface name="velocity"/>
+            </joint>
+            <joint name="finger_joint1">
+                <command_interface name="position"/>
+                <state_interface name="position">
+                  <param name="initial_value">${initial_positions['finger_joint1']}</param>
+                </state_interface>
+                <state_interface name="velocity"/>
+            </joint>
+        </ros2_control>
+    </xacro:macro>
 </robot>

File: mybot/config/six_arm.urdf.xacro (robot description, xacro)
@@ -3,5 +3,5 @@
     <xacro:arg name="initial_positions_file" default="initial_positions.yaml" />
     <!-- Import six_arm urdf file -->
-    <xacro:include filename="$(find mybot_description)/urdf/arm.xacro" />
+    <xacro:include filename="$(find mybot_description)/urdf/originbot_with_arm.xacro" />
     <!-- Import control_xacro -->
     <xacro:include filename="six_arm.ros2_control.xacro" />
